File: sstv-encoder/sstv-encoder.kicad_pcb (KiCad board)
At the start: 2 copper layers, 18 parts, among them U1 ANTENNA_CONN, U2 LM386

Commit message: update schematic
Parts:
- added Alt1: AltlMU-10, sstv-encoder:AltIMU-10, F.Cu at (131.8, 90.9)
- added C10: 10uF, Capacitor_THT:CP_Radial_D5.0mm_P2.50mm, F.Cu at (128.7, 174.5)
- added C11: 10uF, Capacitor_THT:CP_Radial_D5.0mm_P2.50mm, F.Cu at (97.3, 172.1)
- added C9: 1uF, Capacitor_THT:CP_Radial_D5.0mm_P2.50mm, F.Cu at (268.7, 201.6)
- added RV2: 10K, Potentiometer_THT:Potentiometer_Piher_PT-10-V10_Vertical, F.Cu at (234.2, 204.3)
- added U3: Adafruit_GPS_MTK3339, sstv-encoder:Adafruit_GPS, F.Cu at (126.7, 62.9)
- added U4: TL082, Package_DIP:DIP-8-16_W7.62mm, F.Cu at (249.8, 193.5)
- added U5: DG419LDJ, Package_DIP:DIP-8_W7.62mm, F.Cu at (262.6, 169.6)
- added U6: LTC1044, Package_DIP:DIP-8_W7.62mm, F.Cu at (109.9, 169.3)
- RV1: footprint Potentiometer_SMD:Potentiometer_Bourns_3214J_Horizontal -> Potentiometer_THT:Potentiometer_Piher_PT-10-V10_Vertical
- moved C6 207.6 mm to (311.1, 50.3)
- moved C4 207.4 mm to (311.2, 40.4)
- moved R1 171.8 mm to (168.7, 266.2)
- moved U2 169.4 mm to (166.9, 234.4)
- moved C5 168.7 mm to (198.0, 258.9)
- moved RV1 168.5 mm to (131.1, 262.1)
- moved U1 161.8 mm to (302.1, 29.5)
- moved VHF_TRANS1 159.2 mm to (283.6, 52.7)
- moved R2 157.1 mm to (191.4, 249.5)
- moved C7 154.4 mm to (197.1, 269.7)
- moved C8 139.3 mm to (311.9, 58.5)
- moved SD1 109.5 mm to (87.4, 69.3), turned to 180 degrees
- moved CAM1 80.1 mm to (191.8, 1.31), turned to 90 degrees
- moved C3 78.9 mm to (91.1, 93.3)
- moved C2 77.7 mm to (91.1, 98.0)
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Connections:
- DUE1 pad 10: (no net) -> /RX_DRA
- DUE1 pad 11: (no net) -> /TX_GPS
- DUE1 pad 12: (no net) -> /RX_GPS
- DUE1 pad 13: (no net) -> /CS_SD
- DUE1 pad 14: (no net) -> /W_CLK_ADS
- DUE1 pad 15: (no net) -> /FQ_UD_ADS
- DUE1 pad 16: (no net) -> /DATA_ADS
- DUE1 pad 17: (no net) -> /RESET_ADS
- DUE1 pad 18: (no net) -> /PD_DRA
- DUE1 pad 19: (no net) -> /PTT_DRA
- DUE1 pad 20: (no net) -> /POW_DRA
- DUE1 pad 21: (no net) -> /AF_APRS
- DUE1 pad 22: (no net) -> /MUX_SL
- DUE1 pad 23: (no net) -> /SDA_IMU
- DUE1 pad 24: (no net) -> /SCL_IMU
- DUE1 pad 5: (no net) -> /MOSI_SD
- DUE1 pad 6: (no net) -> /SCK_SD
- DUE1 pad 7: (no net) -> /TX_CAM
- DUE1 pad 8: (no net) -> /RX_CAM
- DUE1 pad 9: (no net) -> /TX_DRA
- R1 pad 2: /ZOUT_ADS -> /AF_MUX
- U1 pad 1: (no net) -> Net-(U1-Pad1)
- U1 pad 2: (no net) -> GNDREF
- VHF_TRANS1 pad 12: Net-(U1-Pad~) -> Net-(U1-Pad1)
Routing:
- net /MOSI_SD: track 0.00 -> 60.5 mm
- net +3V3: track 0.00 -> 54.9 mm
- net /SDA_IMU: track 0.00 -> 52.9 mm
- net /RESET_ADS: track 0.00 -> 50.7 mm
- net /DATA_ADS: track 0.00 -> 49.9 mm
- net /FQ_UD_ADS: track 0.00 -> 49.2 mm
- net /W_CLK_ADS: track 0.00 -> 48.5 mm
- net /SCL_IMU: track 0.00 -> 46.8 mm
- net /MISO_SD: track 0.00 -> 44.9 mm
- net /SCK_SD: track 0.00 -> 25.8 mm
- net GNDREF: track 0.00 -> 17.2 mm
- net /RX_GPS: track 0.00 -> 7.95 mm
- net /TX_GPS: track 0.00 -> 7.95 mm
- net /CS_SD: track 0.00 -> 2.15 mm

Commit message: finish pcb
Parts:
- added G***: LOGO, Logo:logo, F.Cu at (53.3, 52.1)
- moved U1 263.8 mm to (55.0, 121.9)
- moved C9 255.7 mm to (53.6, 63.2), turned to 180 degrees
- moved U5 235.9 mm to (48.5, 70.6)
- moved U4 230.0 mm to (61.6, 61.5)
- moved RV2 217.0 mm to (48.1, 92.7)
- moved VHF_TRANS1 209.3 mm to (85.1, 118.8)
- moved R1 204.4 mm to (50.1, 99.7)
- moved C4 186.3 mm to (131.9, 90.9)
- moved C5 184.9 mm to (131.2, 86.4)
- moved C7 184.4 mm to (132.2, 97.2)
- moved C6 176.0 mm to (141.5, 97.2)
- moved C8 173.5 mm to (141.5, 90.9)
- moved U2 172.9 mm to (78.2, 85.9)
- moved RV1 172.6 mm to (48.1, 110.8)
- moved R2 170.8 mm to (140.3, 86.6)
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Connections:
- U3 pad 8: +3V3 -> +5V
Routing:
- net +5V: track 0.00 -> 168.8 mm, vias 0 -> 2
- net /RX_DRA: track 0.00 -> 151.0 mm, vias 0 -> 2
- net /TX_DRA: track 0.00 -> 137.1 mm, vias 0 -> 2
- net /POW_DRA: track 0.00 -> 117.4 mm
- net /PD_DRA: track 0.00 -> 108.1 mm
- net /MUX_SL: track 0.00 -> 106.1 mm, vias 0 -> 2
- net /ZOUT_ADS: track 0.00 -> 101.5 mm
- net /PTT_DRA: track 0.00 -> 100.4 mm, vias 0 -> 1
- net Net-(C5-Pad1): track 0.00 -> 85.4 mm, vias 0 -> 2
- net /AF_APRS: track 0.00 -> 77.0 mm
- net /CS_SD: track 2.15 -> 72.4 mm, vias 0 -> 1
- net /RX_CAM: track 0.00 -> 47.1 mm, vias 0 -> 1
- net /AF_IN: track 0.00 -> 44.6 mm, vias 0 -> 1
- net /TX_CAM: track 0.00 -> 39.8 mm
- net /MOSI_SD: track 60.5 -> 24.4 mm
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- added copper zone on B.Cu, net GNDREF
- added copper zone on F.Cu, net GNDREF
Other:
- board outline added: 114 x 89 mm
- board text added: "+"
- board text added: "RadioClub E.I.T 2020 Fran Acién | Pablo Alvarez | David Arias | Dani Kohler Ke pasa ente | Mamado picado | Nostalgico | Cuando unos patos"

Commit message: fix error
Parts:
- moved RV1 13.4 mm to (49.5, 124.1)
- moved U1 13.0 mm to (58.3, 109.3)
Routing:
- net Net-(RV1-Pad2): track 31.7 -> 50.6 mm
- net Net-(U1-Pad1): track 26.0 -> 13.2 mm
- net Net-(R1-Pad1): track 14.2 -> 26.4 mm
- net (no net): vias 0 -> 8
Changed lines of the file:
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@@
     (thickness 1.6)
     (drawings 20)
-    (tracks 382)
+    (tracks 385)
     (zones 0)
     (modules 28)
@@
   )
   (setup
-    (last_trace_width 0.5)
+    (last_trace_width 0.7)
     (user_trace_width 0.5)
     (user_trace_width 0.7)
     (user_trace_width 1)
+    (user_trace_width 1.4)
     (trace_clearance 0.2)
     (zone_clearance 0.508)
@@
   )
   (module sstv-encoder:SMA_conn (layer F.Cu)
-    (at 55.0418 121.9073)
+    (at 58.2676 109.2835)
     (fp_text reference U1 (at -0.1016 5.461) (layer F.SilkS)
       (effects (font (size 1 1) (thickness 0.15)))
@@
   )
   (module Potentiometer_THT:Potentiometer_Piher_PT-10-V10_Vertical (layer F.Cu)
-    (at 48.133 110.7821)
+    (at 49.5046 124.1425)
     (descr "Potentiometer, vertical, Piher PT-10-V10, http://www.piher-nacesa.com/pdf/12-PT10v03.pdf")
     (tags "Potentiometer vertical Piher PT-10-V10")
@@
   (gr_circle (center 75.6294 80.8025) (end 76.8794 80.8025) (layer Edge.Cuts) (width 0.12))
   (gr_circle (center 75.6294 60.8025) (end 76.8794 60.8025) (layer Edge.Cuts) (width 0.12))
+  (via (at 69.1896 107.7595) (size 0.8) (drill 0.4) (layers F.Cu B.Cu) (net 0))
+  (via (at 67.7926 107.7595) (size 0.8) (drill 0.4) (layers F.Cu B.Cu) (net 0))
+  (via (at 66.5226 107.7595) (size 0.8) (drill 0.4) (layers F.Cu B.Cu) (net 0))
+  (via (at 65.1256 107.7595) (size 0.8) (drill 0.4) (layers F.Cu B.Cu) (net 0))
+  (via (at 63.8556 107.7595) (size 0.8) (drill 0.4) (layers F.Cu B.Cu) (net 0))
+  (via (at 62.7126 107.7595) (size 0.8) (drill 0.4) (layers F.Cu B.Cu) (net 0))
+  (via (at 62.8396 110.6805) (size 0.8) (drill 0.4) (layers F.Cu B.Cu) (net 0))
+  (via (at 64.1096 110.6805) (size 0.8) (drill 0.4) (layers F.Cu B.Cu) (net 0))
   (segment (start 93.6352 93.3704) (end 93.5717 93.3069) (width 0.7) (layer F.Cu) (net 1))
   (segment (start 93.5717 87.63) (end 93.5971 87.6046) (width 0.7) (layer F.Cu) (net 1))
@@
   (segment (start 135.8138 56.8325) (end 136.062299 56.584001) (width 0.5) (layer F.Cu) (net 11))
   (segment (start 123.317 56.8325) (end 135.8138 56.8325) (width 0.5) (layer F.Cu) (net 11))
-  (segment (start 50.814199 100.356899) (end 50.864999 100.356899) (width 0.7) (layer F.Cu) (net 12))
-  (segment (start 50.1142 99.6569) (end 50.814199 100.356899) (width 0.7) (layer F.Cu) (net 12))
-  (segment (start 50.864999 100.356899) (end 53.0606 102.5525) (width 0.7) (layer F.Cu) (net 12))
-  (segment (start 53.0606 102.5525) (end 53.0606 106.4133) (width 0.7) (layer F.Cu) (net 12))
-  (segment (start 53.0606 106.4133) (end 48.7426 110.7313) (width 0.7) (layer F.Cu) (net 12))
-  (segment (start 48.7426 110.7313) (end 48.7426 110.7821) (width 0.7) (layer F.Cu) (net 12))
+  (segment (start 50.1142 99.6569) (end 50.1142 115.1001) (width 0.7) (layer F.Cu) (net 12))
+  (segment (start 50.1142 115.1001) (end 52.5526 117.5385) (width 0.7) (layer F.Cu) (net 12))
+  (segment (start 52.5526 117.5385) (end 52.5526 121.4755) (width 0.7) (layer F.Cu) (net 12))
+  (segment (start 52.5526 121.4755) (end 50.0126 124.0155) (width 0.7) (layer F.Cu) (net 12))
   (segment (start 66.3702 70.5993) (end 56.1594 70.5993) (width 1) (layer F.Cu) (net 13))
   (segment (start 94.3102 70.6501) (end 66.421 70.6501) (width 1) (layer F.Cu) (net 13))
@@
   (segment (start 126.5682 105.1941) (end 126.5682 95.3389) (width 1) (layer F.Cu) (net 13))
   (segment (start 77.8002 90.9701) (end 78.3082 90.9701) (width 1) (layer F.Cu) (net 14))
-  (segment (start 59.302999 101.593301) (end 64.3382 96.5581) (width 1) (layer F.Cu) (net 14))
-  (segment (start 59.302999 107.112101) (end 59.302999 101.593301) (width 1) (layer F.Cu) (net 14))
-  (segment (start 58.133 108.2821) (end 59.302999 107.112101) (width 1) (layer F.Cu) (net 14))
-  (segment (start 64.3382 96.5581) (end 73.9394 96.5581) (width 1) (layer F.Cu) (net 14))
-  (segment (start 73.9394 96.5581) (end 73.9902 96.5581) (width 1) (layer F.Cu) (net 14))
-  (segment (start 73.9902 96.5581) (end 76.4286 94.1197) (width 1) (layer F.Cu) (net 14))
-  (segment (start 76.4286 94.1197) (end 76.4286 92.5957) (width 1) (layer F.Cu) (net 14))
-  (segment (start 76.4286 92.5957) (end 78.0542 90.9701) (width 1) (layer F.Cu) (net 14))
+  (segment (start 59.5046 121.6425) (end 53.0606 115.1985) (width 0.7) (layer F.Cu) (net 14))
+  (segment (start 53.0606 115.1985) (end 53.0606 105.3465) (width 0.7) (layer F.Cu) (net 14))
+  (segment (start 61.849 96.5581) (end 64.3382 96.5581) (width 0.7) (layer F.Cu) (net 14))
+  (segment (start 53.0606 105.3465) (end 61.849 96.5581) (width 0.7) (layer F.Cu) (net 14))
+  (segment (start 64.3382 96.5581) (end 73.152 96.5581) (width 0.7) (layer F.Cu) (net 14))
+  (segment (start 73.152 96.5581) (end 76.1746 93.5355) (width 0.7) (layer F.Cu) (net 14))
+  (segment (start 76.1746 93.5355) (end 76.1746 92.3925) (width 0.7) (layer F.Cu) (net 14))
+  (segment (start 76.1746 92.3925) (end 77.5716 90.9955) (width 0.7) (layer F.Cu) (net 14))
   (via (at 153.9494 86.0425) (size 0.8) (drill 0.4) (layers F.Cu B.Cu) (net 15))
   (segment (start 153.9494 86.0425) (end 153.9494 94.9833) (width 0.25) (layer F.Cu) (net 15))
@@
   (segment (start 59.563 88.8365) (end 57.9882 90.4113) (width 0.7) (layer F.Cu) (net 61))
   (segment (start 61.595 63.9953) (end 61.595 61.3029) (width 0.5) (layer F.Cu) (net 67))
-  (segment (start 55.0418 121.9073) (end 59.2582 121.9073) (width 1) (layer F.Cu) (net 70))
-  (segment (start 59.2582 121.9073) (end 63.2206 117.9449) (width 1) (layer F.Cu) (net 70))
-  (segment (start 63.2206 117.9449) (end 63.2206 111.0361) (width 1) (layer F.Cu) (net 70))
-  (segment (start 63.2206 111.0361) (end 65.8622 108.3945) (width 1) (layer F.Cu) (net 70))
-  (segment (start 65.8622 108.3945) (end 71.3486 108.3945) (width 1) (layer F.Cu) (net 70))
+  (segment (start 71.7146 109.3085) (end 58.6236 109.3085) (width 1.4) (layer F.Cu) (net 70))
+  (segment (start 58.6236 109.3085) (end 58.5216 109.4105) (width 1.4) (layer F.Cu) (net 70))
+  (zone (net 1) (net_name GNDREF) (layer F.Cu) (hatch edge 0.508)
+    (connect_pads (clearance 0.508))
+    (min_thickness 0.254)
+    (fill yes (arc_segments 32) (thermal_gap 0.508) (thermal_bridge_width 0.508))
+    (polygon
+      (pts
+        (xy 160.8836 135.6995) (xy 43.0276 135.4455) (xy 43.0276 43.1165) (xy 161.0106 43.1165)
+      )
+    )
+  )
   (zone (net 1) (net_name GNDREF) (layer B.Cu) (hatch edge 0.508)
     (connect_pads (clearance 0.508))
@@
     (polygon
       (pts
-        (xy 159.4866 42.7355) (xy 160.1216 134.8105) (xy 42.6466 135.3185) (xy 43.2816 42.4815)
+        (xy 161.1376 136.3345) (xy 42.7736 136.3345) (xy 42.7736 42.7355) (xy 160.8836 42.7355)
       )
     )
-  )
-  (zone (net 1) (net_name GNDREF) (layer F.Cu) (hatch edge 0.508)
-    (connect_pads (clearance 0.508))
-    (min_thickness 0.254)
-    (fill yes (arc_segments 32) (thermal_gap 0.508) (thermal_bridge_width 0.508))
-    (polygon
-      (pts
-        (xy 159.8676 42.9895) (xy 160.6296 134.9375) (xy 43.2816 135.4455) (xy 43.0276 42.2275)
-      )
-    )

Commit message: fix footprint error
Parts:
- U4: footprint Package_DIP:DIP-8-16_W7.62mm -> Package_DIP:DIP-8_W7.62mm
- moved U4 12.8 mm to (63.5, 74.1)
Connections:
- U5 pad 2: /AF_APRS -> /AF_APRS_NORM
Routing:
- net /AF_APRS_NORM: track 2.69 -> 24.7 mm, vias 0 -> 1
- net /AF_APRS: track 77.0 -> 66.2 mm
- net Net-(RV2-Pad2): track 15.2 -> 13.6 mm
- net /AF_MUX: track 33.5 -> 32.3 mm
